File: Atharva-EPS.kicad_pcb (KiCad board)
At the start: 4 copper layers, 86.3 x 94.9 mm, 0 parts

Commit message: Placed footprints on PCB, improvements on schematic
Parts:
- added BT101: Battery_Cell, 254TR:BAT_254TR, F.Cu at (76.0, 64.3)
- added BT102: Battery_Cell, 254TR:BAT_254TR, F.Cu at (76.1, 86.9)
- added BT103: Battery_Cell, 254TR:BAT_254TR, F.Cu at (76.5, 135.1)
- added BT104: Battery_Cell, 254TR:BAT_254TR, F.Cu at (77.3, 109.9)
- added C101: 0.1uF, Capacitor_SMD:C_0805_2012Metric, F.Cu at (106.0, 91.5)
- added C102: 0.1uF, Capacitor_SMD:C_0805_2012Metric, F.Cu at (105.8, 86.6)
- added C103: 6.8uF, Capacitor_SMD:C_0805_2012Metric, F.Cu at (103.7, 81.4)
- added C104: 6.8uF, Capacitor_SMD:C_0805_2012Metric, F.Cu at (108.2, 77.9)
- added C105: 0.01uF, Capacitor_SMD:C_0805_2012Metric, F.Cu at (125.0, 78.7)
- added C106: 0.1uF, Capacitor_SMD:C_0805_2012Metric, F.Cu at (134.5, 85.1)
- added C107: 0.1uF, Capacitor_SMD:C_0805_2012Metric, F.Cu at (120.4, 94.1)
- added C108: 10uF, Capacitor_SMD:C_0805_2012Metric, F.Cu at (93.0, 117.8)
- added C109: 10uF, Capacitor_SMD:C_0805_2012Metric, F.Cu at (97.8, 136.6)
- added C110: 10uF, Capacitor_SMD:C_0805_2012Metric, F.Cu at (100.2, 104.0)
- added C111: 1uF, Capacitor_SMD:C_0805_2012Metric, F.Cu at (106.3, 116.3)
- added C112: 1uF, Capacitor_SMD:C_0805_2012Metric, F.Cu at (112.8, 136.4)
- added C113: 1uF, Capacitor_SMD:C_0805_2012Metric, F.Cu at (114.1, 102.4)
- added C114: 10uF, Capacitor_SMD:C_0805_2012Metric, F.Cu at (121.9, 121.5)
- added C115: 10uF, Capacitor_SMD:C_0805_2012Metric, F.Cu at (117.7, 141.6)
- added C116: 10uF, Capacitor_SMD:C_0805_2012Metric, F.Cu at (111.6, 108.7)
- added C117: 10uF, Capacitor_SMD:C_0805_2012Metric, F.Cu at (126.5, 136.6)
- added C118: 10uF, Capacitor_SMD:C_0805_2012Metric, F.Cu at (127.3, 116.2)
- added C119: 10uF, Capacitor_SMD:C_0805_2012Metric, F.Cu at (128.9, 100.7)
- added C120: 1uF, Capacitor_SMD:C_0805_2012Metric, F.Cu at (141.2, 135.7)
- added C121: 1uF, Capacitor_SMD:C_0805_2012Metric, F.Cu at (140.5, 113.4)
- added C122: 1uF, Capacitor_SMD:C_0805_2012Metric, F.Cu at (144.2, 99.2)
- added C123: 10uF, Capacitor_SMD:C_0805_2012Metric, F.Cu at (149.7, 140.9)
- added C124: 10uF, Capacitor_SMD:C_0805_2012Metric, F.Cu at (150.3, 119.3)
- added C125: 10uF, Capacitor_SMD:C_0805_2012Metric, F.Cu at (147.4, 108.5)
- added D101: 1N5817, Diode_THT:D_DO-41_SOD81_P10.16mm_Horizontal, F.Cu at (111.2, 68.9)
- added D102: D_Schottky, Diode_SMD:D_1210_3225Metric, F.Cu at (129.2, 72.5)
- added D103: D_Schottky, Diode_SMD:D_1210_3225Metric, F.Cu at (93.9, 113.4)
- added D104: D_Schottky, Diode_SMD:D_1210_3225Metric, F.Cu at (98.5, 132.0)
- added D105: D_Schottky, Diode_SMD:D_1210_3225Metric, F.Cu at (95.4, 99.4)
- added D106: D_Schottky, Diode_SMD:D_1210_3225Metric, F.Cu at (115.9, 116.5)
- added D107: D, Diode_SMD:D_1210_3225Metric, F.Cu at (110.9, 116.6)
- added D108: D_Schottky, Diode_SMD:D_1210_3225Metric, F.Cu at (115.9, 130.5)
- added D109: D, Diode_SMD:D_1210_3225Metric, F.Cu at (117.1, 136.6)
- added D110: D_Schottky, Diode_SMD:D_1210_3225Metric, F.Cu at (114.3, 97.7)
- added D111: D, Diode_SMD:D_1210_3225Metric, F.Cu at (119.3, 102.6)
- added D112: D_Schottky, Diode_SMD:D_1210_3225Metric, F.Cu at (100.9, 111.0)
- added D113: D_Schottky, Diode_SMD:D_1210_3225Metric, F.Cu at (123.0, 130.9)
- added D114: D_Schottky, Diode_SMD:D_1210_3225Metric, F.Cu at (124.8, 100.4)
- added D115: D_Schottky, Diode_SMD:D_1210_3225Metric, F.Cu at (132.1, 130.3)
- added D116: D_Schottky, Diode_SMD:D_1210_3225Metric, F.Cu at (126.3, 111.8)
- added D117: D_Schottky, Diode_SMD:D_1210_3225Metric, F.Cu at (129.3, 94.9)
- added D118: D_Schottky, Diode_SMD:D_1210_3225Metric, F.Cu at (142.1, 130.6)
- added D119: D, Diode_SMD:D_1210_3225Metric, F.Cu at (145.5, 136.3)
- added D120: D_Schottky, Diode_SMD:D_1210_3225Metric, F.Cu at (145.1, 114.1)
- added D121: D, Diode_SMD:D_1210_3225Metric, F.Cu at (141.6, 120.2)
- added D122: D_Schottky, Diode_SMD:D_1210_3225Metric, F.Cu at (145.0, 94.0)
- added D123: D, Diode_SMD:D_1210_3225Metric, F.Cu at (148.6, 99.4)
- added D124: D_Schottky, Diode_SMD:D_1210_3225Metric, F.Cu at (147.6, 130.2)
- added D125: D_Schottky, Diode_SMD:D_1210_3225Metric, F.Cu at (152.1, 113.3)
- added D126: D_Schottky, Diode_SMD:D_1210_3225Metric, F.Cu at (153.7, 97.6)
- added D127: D, Diode_SMD:D_0805_2012Metric_Pad1.15x1.40mm_HandSolder, F.Cu at (94.1, 121.8)
- added D128: D, Diode_SMD:D_0805_2012Metric_Pad1.15x1.40mm_HandSolder, F.Cu at (101.4, 140.4)
- added D129: D, Diode_SMD:D_0805_2012Metric_Pad1.15x1.40mm_HandSolder, F.Cu at (95.5, 105.4)
- added D130: D, Diode_SMD:D_0805_2012Metric_Pad1.15x1.40mm_HandSolder, F.Cu at (136.6, 142.0)
- added D131: D, Diode_SMD:D_0805_2012Metric_Pad1.15x1.40mm_HandSolder, F.Cu at (127.2, 120.4)
- added D132: D, Diode_SMD:D_0805_2012Metric_Pad1.15x1.40mm_HandSolder, F.Cu at (138.1, 108.0)
- added H101: MountingHole, MountingHole:MountingHole_3.2mm_M3_ISO7380_Pad_TopBottom, F.Cu at (93.6, 55.7)
- added H102: MountingHole, MountingHole:MountingHole_3.2mm_M3_ISO7380_Pad_TopBottom, F.Cu at (172.0, 55.5)
- added H103: MountingHole, MountingHole:MountingHole_3.2mm_M3_ISO7380_Pad_TopBottom, F.Cu at (93.6, 142.0)
- added H104: MountingHole, MountingHole:MountingHole_3.2mm_M3_ISO7380_Pad_TopBottom, F.Cu at (172.2, 141.7)
- added J101: Conn_01x02_Female, Connector_Hirose:Hirose_DF13-02P-1.25DSA_1x02_P1.25mm_Vertical, F.Cu at (92.5, 78.3)
- added J102: Conn_01x02_Female, Connector_Hirose:Hirose_DF13-02P-1.25DSA_1x02_P1.25mm_Vertical, F.Cu at (92.5, 73.2)
- added J103: Conn_01x02_Female, Connector_Hirose:Hirose_DF13-02P-1.25DSA_1x02_P1.25mm_Vertical, F.Cu at (92.4, 83.5)
- added J104: Conn_01x02_Female, Connector_Hirose:Hirose_DF13-02P-1.25DSA_1x02_P1.25mm_Vertical, F.Cu at (92.3, 89.0)
- added J105: Conn_02x26_Odd_Even, Connector_PinSocket_2.54mm:PinSocket_2x26_P2.54mm_Vertical, F.Cu at (102.3, 54.4)
- added J106: Conn_02x26_Odd_Even, Connector_PinSocket_2.54mm:PinSocket_2x26_P2.54mm_Vertical, F.Cu at (102.3, 60.8)
- added J107: Conn_01x05_Female, Connector_Hirose:Hirose_DF63-5P-3.96DSA_1x05_P3.96mm_Vertical, F.Cu at (43.3, 60.1)
- added J108: Conn_01x05_Female, Connector_Hirose:Hirose_DF63-5P-3.96DSA_1x05_P3.96mm_Vertical, F.Cu at (42.6, 122.1)
- added J109: Conn_01x05_Female, Connector_Hirose:Hirose_DF63-5P-3.96DSA_1x05_P3.96mm_Vertical, F.Cu at (42.4, 84.7)
- added J110: Conn_01x05_Female, Connector_Hirose:Hirose_DF63-5P-3.96DSA_1x05_P3.96mm_Vertical, F.Cu at (42.9, 96.4)
- added J111: Conn_01x05_Female, Connector_Hirose:Hirose_DF63-5P-3.96DSA_1x05_P3.96mm_Vertical, F.Cu at (42.6, 108.3)
- added J112: Conn_01x05_Female, Connector_Hirose:Hirose_DF63-5P-3.96DSA_1x05_P3.96mm_Vertical, F.Cu at (42.9, 72.5)
- added JP107: Jumper, Jumper:SolderJumper-3_P1.3mm_Open_RoundedPad1.0x1.5mm, F.Cu at (92.7, 68.1)
- added L101: 10uH, Inductor_SMD:L_1210_3225Metric, F.Cu at (113.1, 122.5)
- added L102: 10uH, Inductor_SMD:L_1210_3225Metric, F.Cu at (109.1, 130.8)
- added L103: 10uH, Inductor_SMD:L_1210_3225Metric, F.Cu at (109.3, 97.3)
- added L104: 10uH, Inductor_SMD:L_1210_3225Metric, F.Cu at (152.8, 136.1)
- added L105: 10uH, Inductor_SMD:L_1210_3225Metric, F.Cu at (136.8, 120.2)
- added L106: 10uH, Inductor_SMD:L_1210_3225Metric, F.Cu at (140.2, 96.6)
- added Q101: P-MOSFET-SOT23-3, TSM2307CX:SOT23-3, F.Cu at (105.5, 69.0)
- added Q102: 2N3906, Package_TO_SOT_THT:TO-92_Inline, F.Cu at (152.8, 71.1)
- added Q103: 2N3906, Package_TO_SOT_THT:TO-92_Inline, F.Cu at (159.9, 79.9)
- added Q104: IRLML2060, Package_TO_SOT_SMD:SOT-23, F.Cu at (141.4, 78.0)
- added Q105: IRLML2060, Package_TO_SOT_SMD:SOT-23, F.Cu at (124.0, 88.6)
- added Q106: IRLML2060, Package_TO_SOT_SMD:SOT-23, F.Cu at (149.3, 79.5)
- added Q107: IRLML2060, Package_TO_SOT_SMD:SOT-23, F.Cu at (149.1, 86.3)
- added R101: 1M, Resistor_SMD:R_0805_2012Metric, F.Cu at (158.4, 75.6)
- added R102: 510k, Resistor_SMD:R_0805_2012Metric, F.Cu at (147.3, 72.2)
- added R103: 1M, Resistor_SMD:R_0805_2012Metric, F.Cu at (163.2, 86.2)
- added R104: 510k, Resistor_SMD:R_0805_2012Metric, F.Cu at (158.6, 86.3)
- added R105: 1k, Resistor_SMD:R_0805_2012Metric, F.Cu at (125.1, 83.1)
- added R106: 1k, Resistor_SMD:R_0805_2012Metric, F.Cu at (110.9, 82.6)
- added R107: 1k, Resistor_SMD:R_0805_2012Metric, F.Cu at (129.7, 83.0)
- added R108: 1k, Resistor_SMD:R_0805_2012Metric, F.Cu at (110.9, 87.1)
- added R109: 470, Resistor_SMD:R_0805_2012Metric, F.Cu at (138.6, 85.4)
- added R110: 51, Resistor_SMD:R_0805_2012Metric, F.Cu at (143.6, 83.6)
- added R111: 470, Resistor_SMD:R_0805_2012Metric, F.Cu at (121.0, 82.8)
- added R112: 51, Resistor_SMD:R_0805_2012Metric, F.Cu at (128.0, 88.0)
- added R113: 530k, Resistor_SMD:R_0805_2012Metric, F.Cu at (99.3, 115.7)
- added R114: 100k, Resistor_SMD:R_0805_2012Metric, F.Cu at (97.8, 119.5)
- added R115: 530k, Resistor_SMD:R_0805_2012Metric, F.Cu at (104.0, 132.6)
- added R116: 100k, Resistor_SMD:R_0805_2012Metric, F.Cu at (104.2, 136.5)
- added R117: 530k, Resistor_SMD:R_0805_2012Metric, F.Cu at (100.5, 100.0)
- added R118: 100k, Resistor_SMD:R_0805_2012Metric, F.Cu at (105.1, 103.5)
- added R119: 542k, Resistor_SMD:R_0805_2012Metric, F.Cu at (108.3, 121.0)
- added R120: 542k, Resistor_SMD:R_0805_2012Metric, F.Cu at (113.7, 142.7)
- added R121: 542k, Resistor_SMD:R_0805_2012Metric, F.Cu at (115.8, 106.7)
- added R122: 459k, Resistor_SMD:R_0805_2012Metric, F.Cu at (109.0, 125.3)
- added R123: 459k, Resistor_SMD:R_0805_2012Metric, F.Cu at (108.7, 142.0)
- added R124: 459k, Resistor_SMD:R_0805_2012Metric, F.Cu at (106.4, 108.7)
- added R125: 0.05, Resistor_SMD:R_0805_2012Metric, F.Cu at (117.4, 122.1)
- added R126: 0.05, Resistor_SMD:R_0805_2012Metric, F.Cu at (121.9, 137.6)
- added R127: 0.05, Resistor_SMD:R_0805_2012Metric, F.Cu at (120.3, 107.8)
- added R128: 530k, Resistor_SMD:R_0805_2012Metric, F.Cu at (131.2, 134.9)
- added R129: 100k, Resistor_SMD:R_0805_2012Metric, F.Cu at (131.0, 138.8)
- added R130: 530k, Resistor_SMD:R_0805_2012Metric, F.Cu at (131.5, 112.4)
- added R131: 100k, Resistor_SMD:R_0805_2012Metric, F.Cu at (132.1, 116.3)
- added R132: 530k, Resistor_SMD:R_0805_2012Metric, F.Cu at (133.8, 100.6)
- added R133: 100k, Resistor_SMD:R_0805_2012Metric, F.Cu at (133.8, 104.4)
- added R134: 542k, Resistor_SMD:R_0805_2012Metric, F.Cu at (141.5, 142.0)
- added R135: 542k, Resistor_SMD:R_0805_2012Metric, F.Cu at (151.8, 123.6)
- added R136: 542k, Resistor_SMD:R_0805_2012Metric, F.Cu at (146.5, 103.7)
- added R137: 459k, Resistor_SMD:R_0805_2012Metric, F.Cu at (154.1, 143.0)
- added R138: 459k, Resistor_SMD:R_0805_2012Metric, F.Cu at (146.9, 123.6)
- added R139: 459k, Resistor_SMD:R_0805_2012Metric, F.Cu at (142.8, 107.9)
- added R140: 0.05, Resistor_SMD:R_0805_2012Metric, F.Cu at (145.3, 141.9)
- added R141: 0.05, Resistor_SMD:R_0805_2012Metric, F.Cu at (146.1, 119.5)
- added R142: 0.05, Resistor_SMD:R_0805_2012Metric, F.Cu at (151.1, 104.1)
- added R143: 1M, Resistor_SMD:R_0805_2012Metric, F.Cu at (154.0, 79.4)
- added R144: 1M, Resistor_SMD:R_0805_2012Metric, F.Cu at (154.0, 86.0)
- added U101: MAX1615xUK, Package_TO_SOT_SMD:SOT-23-5, F.Cu at (98.6, 90.2)
- added U102: MAX1615xUK, Package_TO_SOT_SMD:SOT-23-5, F.Cu at (98.7, 83.2)
- added U103: S-8209AXXT, S-8209AAA-T8T1y:SOP65P640X120-8N, F.Cu at (133.3, 79.2)
- added U104: S-8209AXXT, S-8209AAA-T8T1y:SOP65P640X120-8N, F.Cu at (117.4, 87.1)
- added U105: LT3652EDD, Package_DFN_QFN:DFN-12-1EP_3x3mm_P0.45mm_EP1.66x2.38mm, F.Cu at (102.3, 119.5)
- added U106: LT3652EDD, Package_DFN_QFN:DFN-12-1EP_3x3mm_P0.45mm_EP1.66x2.38mm, F.Cu at (108.5, 137.1)
- added U107: LT3652EDD, Package_DFN_QFN:DFN-12-1EP_3x3mm_P0.45mm_EP1.66x2.38mm, F.Cu at (109.6, 103.6)
- added U108: LT3652EDD, Package_DFN_QFN:DFN-12-1EP_3x3mm_P0.45mm_EP1.66x2.38mm, F.Cu at (137.4, 136.5)
- added U109: LT3652EDD, Package_DFN_QFN:DFN-12-1EP_3x3mm_P0.45mm_EP1.66x2.38mm, F.Cu at (136.7, 114.2)
- added U110: LT3652EDD, Package_DFN_QFN:DFN-12-1EP_3x3mm_P0.45mm_EP1.66x2.38mm, F.Cu at (140.4, 102.7)

Commit message: combined all MPPTs into one
Parts:
- removed C108, C109, C114, C115, C117, C118, C119, C123, C124, C125: 10uF, Capacitor_SMD:C_0805_2012Metric
- removed C111, C112, C120, C121, C122: 1uF, Capacitor_SMD:C_0805_2012Metric
- removed D103, D104, D106, D108, D112, D113, D115, D116, D117, D118, D120, D122, D124, D125, D126: D_Schottky, Diode_SMD:D_1210_3225Metric
- removed D107, D109, D119, D121, D123: D, Diode_SMD:D_1210_3225Metric
- removed D127, D128, D130, D131, D132: D, Diode_SMD:D_0805_2012Metric_Pad1.15x1.40mm_HandSolder
- removed L101, L102, L104, L105, L106: 10uH, Inductor_SMD:L_1210_3225Metric
- removed R113, R115, R128, R130, R132: 530k, Resistor_SMD:R_0805_2012Metric
- removed R114, R116, R129, R131, R133: 100k, Resistor_SMD:R_0805_2012Metric
- removed R119, R120, R134, R135, R136: 542k, Resistor_SMD:R_0805_2012Metric
- removed R122, R123, R137, R138, R139: 459k, Resistor_SMD:R_0805_2012Metric
- removed R125, R126, R140, R141, R142: 0.05, Resistor_SMD:R_0805_2012Metric
- removed U105, U106, U108, U109, U110: LT3652EDD, Package_DFN_QFN:DFN-12-1EP_3x3mm_P0.45mm_EP1.66x2.38mm
- added TP101: TestPoint, TestPoint:TestPoint_Pad_1.0x1.0mm, F.Cu at (27.1, 110.0)
- added TP102: TestPoint, TestPoint:TestPoint_Pad_1.0x1.0mm, F.Cu at (27.1, 113.0)
- added TP103: TestPoint, TestPoint:TestPoint_Pad_1.0x1.0mm, F.Cu at (30.1, 110.0)
- added TP104: TestPoint, TestPoint:TestPoint_Pad_1.0x1.0mm, F.Cu at (30.1, 113.0)
- added TP105: TestPoint, TestPoint:TestPoint_Pad_1.0x1.0mm, F.Cu at (33.2, 110.0)
- BT101, BT102, BT103, BT104: footprint 254TR:BAT_254TR -> Battery:BatteryHolder_Keystone_1042_1x18650
- J107, J108, J109, J110, J111, J112: footprint Connector_Hirose:Hirose_DF63-5P-3.96DSA_1x05_P3.96mm_Vertical -> Connector_Hirose:Hirose_DF13-05P-1.25DSA_1x05_P1.25mm_Vertical
- moved BT103 167.8 mm to (231.6, 71.1)
- moved BT101 160.3 mm to (231.6, 25.7)
- moved BT102 160.2 mm to (231.6, 48.4)
- moved BT104 155.2 mm to (231.6, 93.8)
- moved J108 50.1 mm to (63.2, 76.4)
- moved J111 44.1 mm to (73.2, 76.4)
- moved J109 33.6 mm to (73.2, 71.0)
- moved J112 31.7 mm to (73.2, 81.9)
- moved J110 25.0 mm to (63.2, 81.9)
- moved J107 22.7 mm to (63.2, 71.0)
- moved C107 13.3 mm to (132.7, 89.1)
- moved U102 6.81 mm to (98.8, 76.4)
- moved D114 6.22 mm to (119.0, 102.6)
- moved C116 5.70 mm to (106.0, 107.6), turned to 180 degrees
- moved R124 5.49 mm to (101.0, 107.6), turned to 180 degrees
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Connections:
- D105 pad 2: S_1 -> Solar_Out
- D111 pad 1: Net-(C113-Pad2) -> Net-(D111-Pad1)
- J107 pad 1: S_1 -> Solar_Out
- J108 pad 1: S_2 -> Solar_Out
- J109 pad 1: S_3 -> Solar_Out
- J110 pad 1: S_4 -> Solar_Out
- J111 pad 1: S_5 -> Solar_Out
- J112 pad 1: S_6 -> Solar_Out
- L103 pad 2: Net-(L103-Pad2) -> Net-(C113-Pad2)
- R127 pad 1: Net-(L103-Pad2) -> Net-(C113-Pad2)
- U107 pad 10: Net-(L103-Pad2) -> Net-(C113-Pad2)
- U107 pad 11: Net-(C113-Pad2) -> Net-(D111-Pad1)
Other:
- copper layers 4 -> 2
- board text added: "MPPT"

Commit message: Changed the schottky diode logic
Parts:
- removed JP107: Jumper, Jumper:SolderJumper-3_P1.3mm_Open_RoundedPad1.0x1.5mm
- added R113: 0, Resistor_SMD:R_0805_2012Metric, F.Cu at (161.9, 76.7)
- added R114: 0, Resistor_SMD:R_0805_2012Metric, F.Cu at (158.0, 80.6)
- added R115: 0, Resistor_SMD:R_0805_2012Metric, F.Cu at (164.5, 88.6)
- added R116: 0, Resistor_SMD:R_0805_2012Metric, F.Cu at (165.2, 96.6)
- added R119: 0, Resistor_SMD:R_0805_2012Metric, F.Cu at (158.9, 112.5)
- added R120: 0, Resistor_SMD:R_0805_2012Metric, F.Cu at (167.4, 112.5)
- added R122: 280, Resistor_SMD:R_0805_2012Metric, F.Cu at (97.3, 69.5)
- added REF**: OSHW-Logo2_9.8x8mm_SilkScreen, Symbol:OSHW-Logo2_9.8x8mm_SilkScreen, F.Cu at (103.8, 141.6)
- added TP106: TestPoint, TestPoint:TestPoint_Pad_1.0x1.0mm, F.Cu at (168.4, 84.8)
- added TP107: TestPoint, TestPoint:TestPoint_Pad_1.0x1.0mm, F.Cu at (93.3, 118.3)
- added TP108: TestPoint, TestPoint:TestPoint_Pad_1.0x1.0mm, F.Cu at (92.4, 135.9)
- BT101, BT102, BT103: moved to B.Cu
- D129: footprint Diode_SMD:D_0805_2012Metric_Pad1.15x1.40mm_HandSolder -> Diode_SMD:D_1210_3225Metric
- moved TP104 142.0 mm to (171.1, 96.0)
- moved TP105 133.1 mm to (159.0, 66.6)
- moved TP103 126.5 mm to (153.4, 81.6)
- moved TP102 125.0 mm to (136.0, 51.6)
- moved TP101 120.0 mm to (132.0, 51.6)
- moved BT103 111.8 mm to (134.0, 125.6)
- moved BT104 102.7 mm to (134.0, 125.6)
- moved J112 91.7 mm to (141.0, 143.6)
- moved J102 89.3 mm to (174.0, 109.9), turned to 90 degrees
- moved J111 84.3 mm to (124.0, 143.6)
- moved J104 82.9 mm to (174.0, 74.6), turned to 90 degrees
- moved J103 82.0 mm to (174.0, 91.6), turned to 90 degrees
- moved Q102 55.0 mm to (102.6, 93.4)
- moved R101 51.9 mm to (109.0, 91.8), turned to 270 degrees
- moved Q106 51.3 mm to (110.1, 112.6), turned to 270 degrees
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Connections:
- BT101 pad 1: RBF_IN -> Net-(BT101-Pad1)
- BT102 pad 2: Net-(BT102-Pad2) -> A
- BT103 pad 1: RBF_IN -> Net-(BT103-Pad1)
- BT104 pad 1: Net-(BT101-Pad2) -> Net-(BT104-Pad1)
- BT104 pad 2: Net-(BT102-Pad2) -> A
- C102 pad 1: B -> Net-(C102-Pad1)
- C104 pad 1: RBF_IN -> +5V
- C107 pad 2: Net-(BT102-Pad2) -> B
- C116 pad 1: A -> MPPT_OUT
- D102 pad 1: A -> Net-(C102-Pad1)
- D102 pad 2: RBF_IN -> USB_Charge
- D111 pad 2: A -> MPPT_OUT
- D114 pad 2: A -> MPPT_OUT
- D129 pad 1: A -> MPPT_OUT
- J105 pad 25: RBF_IN -> +5V
- J105 pad 26: RBF_IN -> +5V
- Q102 pad 1: RBF_IN -> Net-(Q102-Pad1)
- Q103 pad 1: RBF_IN -> Net-(Q102-Pad1)
- Q105 pad 2: Net-(BT102-Pad2) -> B
- Q107 pad 2: Net-(BT102-Pad2) -> B
- R101 pad 1: RBF_IN -> Net-(Q102-Pad1)
- R103 pad 1: RBF_IN -> Net-(Q102-Pad1)
- R106 pad 2: Net-(BT102-Pad2) -> B
- R108 pad 2: Net-(BT102-Pad2) -> B
- R109 pad 1: RBF_IN -> Net-(Q102-Pad1)
- R110 pad 1: RBF_IN -> Net-(Q102-Pad1)
- R111 pad 1: Net-(BT101-Pad2) -> Net-(R111-Pad1)
- R112 pad 1: Net-(BT101-Pad2) -> Net-(R111-Pad1)
- R121 pad 2: A -> MPPT_OUT
- R127 pad 2: A -> MPPT_OUT
- R144 pad 2: Net-(BT102-Pad2) -> B
- TP101 pad 1: RBF_IN -> +5V
- TP103 pad 1: I2C_DATA -> Net-(C102-Pad1)
- TP104 pad 1: I2C_CLK -> Net-(BT101-Pad2)
- U101 pad 1: B -> Net-(C102-Pad1)
- U101 pad 3: Net-(JP107-Pad1) -> +5V
- U101 pad 4: Net-(JP107-Pad1) -> +5V
- U101 pad 5: B -> Net-(C102-Pad1)
- U104 pad 5: Net-(BT102-Pad2) -> B
- U107 pad 9: A -> MPPT_OUT
Routing:
- net Net-(BT104-Pad1): track 0.00 -> 169.5 mm, vias 0 -> 1
- net Net-(Q102-Pad1): track 0.00 -> 79.5 mm
- net Net-(BT103-Pad1): track 0.00 -> 75.0 mm, vias 0 -> 2
- net Net-(BT101-Pad2): track 0.00 -> 45.9 mm
- net Net-(BT101-Pad1): track 0.00 -> 37.5 mm
- net B: track 0.00 -> 36.1 mm, vias 0 -> 1
- net Net-(C107-Pad1): track 0.00 -> 33.2 mm
- net Net-(C106-Pad1): track 0.00 -> 32.9 mm, vias 0 -> 1
- net Net-(Q103-Pad3): track 0.00 -> 24.8 mm
- net GND: track 0.00 -> 23.9 mm
- net Net-(Q102-Pad3): track 0.00 -> 23.8 mm
- net Net-(R104-Pad2): track 0.00 -> 19.7 mm
- net Net-(R106-Pad1): track 0.00 -> 12.1 mm
- net Net-(Q102-Pad2): track 0.00 -> 11.9 mm
- net Net-(R105-Pad1): track 0.00 -> 11.7 mm
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- added copper zone on F.Cu, net (none)
- added copper zone on In1.Cu, net (none)
- added copper zone on B.Cu, net GND
Other:
- outline, holes or cut-outs redrawn
- copper layers 2 -> 4
- net class Default: clearance 0.2 -> 0.3; trace_width 0.25 -> 0.35
- rule trace_clearance: 0.2 -> 0.3
- board text added: "*"
- board text added: "0"
- board text added: "BMS"
- board text added: "Shitter Diode"
- board text added: "Voltage Regulation"
- board text added: "github.com/ATGr8/CubeSat-EPS"
